File: Asignaciones/Room_Link/_autosave-RELAY.kicad_sch (KiCad schematic)
At the start: 16 parts, among them K1 ADW11, K2 ADW11, K3 ADW11, K4 ADW11, K5 ADW11, U1 ULN2003A

Commit message: Nuevos cambios del Room-Link
Parts:
- R1: value R -> 2.4K
- R2, R3, R4, R5: value R -> 1K
Changed lines of the file:
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@@
       (effects (font (size 1.27 1.27)))
     )
-    (property "Value" "R" (at 142.24 105.41 90)
+    (property "Value" "2.4K" (at 142.24 105.41 90)
       (effects (font (size 1.27 1.27)))
     )
@@
       (effects (font (size 1.27 1.27)))
     )
-    (property "Value" "R" (at 106.68 102.87 90)
+    (property "Value" "1K" (at 106.68 102.87 90)
       (effects (font (size 1.27 1.27)))
     )
@@
       (effects (font (size 1.27 1.27)))
     )
-    (property "Value" "R" (at 190.5 107.95 90)
+    (property "Value" "1K" (at 190.5 107.95 90)
       (effects (font (size 1.27 1.27)))
     )
@@
       (effects (font (size 1.27 1.27)))
     )
-    (property "Value" "R" (at 228.6 110.49 90)
+    (property "Value" "1K" (at 228.6 110.49 90)
       (effects (font (size 1.27 1.27)))
     )
@@
       (effects (font (size 1.27 1.27)))
     )
-    (property "Value" "R" (at 265.43 114.3 90)
-      (effects (font (size 1.27 1.27)))
-    )
+    (property "Value" "1K" (at 265.43 114.3 90)
+      (effects (font (size 1.27 1.27)))
+    )

Commit message: ROOM-LINK update KICAD
Parts:
- K1, K2, K3, K4, K5: footprint Relay_THT:Relay_1P1T_NO_10x24x18.8mm_Panasonic_ADW11xxxxW_THT -> nuevo simbolo:AZ921
Changed lines of the file:
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@@
       (effects (font (size 1.27 1.27)) (justify left))
     )
-    (property "Footprint" "Relay_THT:Relay_1P1T_NO_10x24x18.8mm_Panasonic_ADW11xxxxW_THT" (at 211.455 53.34 0)
+    (property "Footprint" "nuevo simbolo:AZ921" (at 211.455 53.34 0)
       (effects (font (size 1.27 1.27)) hide)
     )
@@
       (effects (font (size 1.27 1.27)) (justify left))
     )
-    (property "Footprint" "Relay_THT:Relay_1P1T_NO_10x24x18.8mm_Panasonic_ADW11xxxxW_THT" (at 127.635 53.34 0)
+    (property "Footprint" "nuevo simbolo:AZ921" (at 127.635 53.34 0)
       (effects (font (size 1.27 1.27)) hide)
     )
@@
       (effects (font (size 1.27 1.27)) (justify left))
     )
-    (property "Footprint" "Relay_THT:Relay_1P1T_NO_10x24x18.8mm_Panasonic_ADW11xxxxW_THT" (at 163.195 53.34 0)
+    (property "Footprint" "nuevo simbolo:AZ921" (at 163.195 53.34 0)
       (effects (font (size 1.27 1.27)) hide)
     )
@@
       (effects (font (size 1.27 1.27)) (justify left))
     )
-    (property "Footprint" "Relay_THT:Relay_1P1T_NO_10x24x18.8mm_Panasonic_ADW11xxxxW_THT" (at 286.385 53.34 0)
+    (property "Footprint" "nuevo simbolo:AZ921" (at 286.385 53.34 0)
       (effects (font (size 1.27 1.27)) hide)
     )
@@
       (effects (font (size 1.27 1.27)) (justify left))
     )
-    (property "Footprint" "Relay_THT:Relay_1P1T_NO_10x24x18.8mm_Panasonic_ADW11xxxxW_THT" (at 248.285 53.34 0)
-      (effects (font (size 1.27 1.27)) hide)
-    )
+    (property "Footprint" "nuevo simbolo:AZ921" (at 248.285 53.34 0)
+      (effects (font (size 1.27 1.27)) hide)
+    )
