File: Asignaciones/Room_Link/CONTROL.kicad_sch (KiCad schematic)
At the start: 0 parts

Commit message: ROOM-LINK update KICAD
Parts:
- added C10, C12: 0.1uF, Capacitor_SMD:C_0805_2012Metric_Pad1.18x1.45mm_HandSolder, symbol Device:C
- added C11: 22 uF, Capacitor_SMD:C_0805_2012Metric_Pad1.18x1.45mm_HandSolder, symbol Device:C
- added D19: LED, LED_SMD:LED_0805_2012Metric_Pad1.15x1.40mm_HandSolder, symbol Device:LED
- added J8: Screw_Terminal_01x06, Connector_PinHeader_2.54mm:PinHeader_2x06_P2.54mm_Vertical_SMD, symbol Connector:Screw_Terminal_01x06
- added J9: Conn_ARM_JTAG_SWD_10, Connector_PinHeader_1.27mm:PinHeader_2x05_P1.27mm_Vertical, symbol Connector:Conn_ARM_JTAG_SWD_10
- added R34: 22k, Resistor_SMD:R_0805_2012Metric_Pad1.20x1.40mm_HandSolder, symbol Device:R
- added R35: 1k, Resistor_SMD:R_0805_2012Metric_Pad1.20x1.40mm_HandSolder, symbol Device:R
- added R36, R37, R38, R39, R40: 100k, Resistor_SMD:R_0805_2012Metric_Pad1.20x1.40mm_HandSolder, symbol Device:R
- added R41: 470, Resistor_SMD:R_0805_2012Metric_Pad1.20x1.40mm_HandSolder, symbol Device:R
- added U5: ESP32-WROOM-32, RF_Module:ESP32-WROOM-32, symbol RF_Module:ESP32-WROOM-32
Connections:
- net COM_RS485_LCD: now also U5.6 (IO34)
- net CON_RS485_eXT: now also U5.7 (IO35)
- net INPUT_1MICRO: now also U5.25 (IO0)
- net INPUT_2MICRO: now also U5.29 (IO5)
- net INPUT_3MICRO: now also U5.26 (IO4)
- net INPUT_4MICRO: now also U5.24 (IO2)
- net RLY_FAN1_MICRO: now also U5.10 (IO25)
- net RLY_FAN2_MICRO: now also U5.11 (IO26)
- net RLY_FAN3_MICRO: now also U5.12 (IO27)
- net RLY_OUT1_MICRO: now also U5.36 (IO22)
- net RLY_OUT2_MICRO: now also U5.37 (IO23)
- net Rx_RS485_eXT: now also U5.34 (RXD0/IO3)
- net Rx_RS485_lcd: now also U5.27 (IO16)
- net Tx_RS485_LCD: now also U5.28 (IO17)
- net Tx_RS485_eXT: now also U5.35 (TXD0/IO1)
- new net: J8.2 (Pin_2), U5.30 (IO18)
- new net: J8.3 (Pin_3), U5.8 (IO32)
- new net: J8.4 (Pin_4), U5.31 (IO19)
- new net: J8.6 (Pin_6), U5.33 (IO21)
- new net: D19.1 (K), U5.9 (IO33)
- new net: D19.2 (A), R41.1
- new net: J9.1 (VTref), R35.2
- new net EN: C10.2, J9.10 (~{RESET}), R34.2, R40.2, U5.3 (EN)
- new net GND: C11.2, C12.2, J8.5 (Pin_5), J9.3 (GND), J9.5 (GND), J9.9 (GNDDetect), U5.1 (GND), U5.15 (GND), U5.38 (GND), U5.39 (GND)
- new net MTCLK: J9.4 (SWDCLK/TCK), R37.2, U5.16 (IO13)
- new net MTD0: J9.6 (SWO/TDO), R38.2, U5.23 (IO15)
- new net MTD1: J9.8 (NC/TDI), R39.2, U5.14 (IO12)
- new net MTM5: U5.13 (IO14)
- new net MTMS: J9.2 (SWDIO/TMS), R36.2
- new net VDD: C10.1, C11.1, C12.1, J8.1 (Pin_1), R34.1, R35.1, R36.1, R37.1, R38.1, R39.1, R40.1, R41.2, U5.2 (VDD)
- no-connect marks 0 -> 9

Commit message: Added nuevos cambios
Parts:
- J8: footprint Connector_PinHeader_2.54mm:PinHeader_2x06_P2.54mm_Vertical_SMD -> Connector_PinHeader_2.54mm:PinHeader_1x06_P2.54mm_Vertical_SMD_Pin1Left
- J9: value Conn_ARM_JTAG_SWD_10 -> JTAG_ ESP32
- R35: value 1k -> 22k
- R36, R37, R38, R39, R40: value 100k -> 10K
Connections:
- net MTM5 is gone; now on net MTMS: U5.13 (IO14)
- net INPUT_1MICRO: now also U5.29 (IO5); no longer U5.25 (IO0)
- net INPUT_2MICRO: now also U5.26 (IO4); no longer U5.29 (IO5)
- net INPUT_3MICRO: now also U5.25 (IO0); no longer U5.26 (IO4)
- net MTCLK renamed MTCK
- net MTD1 renamed MTDI
- no-connect marks 9 -> 10
Other:
- moved on the sheet: R39

Commit message: Place component Added & routing
Parts:
- C10, C11, C12: footprint Capacitor_SMD:C_0805_2012Metric_Pad1.18x1.45mm_HandSolder -> Capacitor_SMD:C_0805_2012Metric
- D19: footprint LED_SMD:LED_0805_2012Metric_Pad1.15x1.40mm_HandSolder -> LED_SMD:LED_0805_2012Metric
- R34, R35, R36, R37, R38, R39, R40, R41: footprint Resistor_SMD:R_0805_2012Metric_Pad1.20x1.40mm_HandSolder -> Resistor_SMD:R_0805_2012Metric
Changed lines of the file:
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@@
       (effects (font (size 1.27 1.27)) (justify left))
     )
-    (property "Footprint" "Resistor_SMD:R_0805_2012Metric_Pad1.20x1.40mm_HandSolder" (at 92.71 98.298 90)
+    (property "Footprint" "Resistor_SMD:R_0805_2012Metric" (at 92.71 98.298 90)
       (effects (font (size 1.27 1.27)) hide)
     )
@@
       (effects (font (size 1.27 1.27)) (justify left))
     )
-    (property "Footprint" "Resistor_SMD:R_0805_2012Metric_Pad1.20x1.40mm_HandSolder" (at 91.44 93.218 90)
+    (property "Footprint" "Resistor_SMD:R_0805_2012Metric" (at 91.44 93.218 90)
       (effects (font (size 1.27 1.27)) hide)
     )
@@
       (effects (font (size 1.27 1.27)) (justify left))
     )
-    (property "Footprint" "Capacitor_SMD:C_0805_2012Metric_Pad1.18x1.45mm_HandSolder" (at 98.7552 46.99 0)
+    (property "Footprint" "Capacitor_SMD:C_0805_2012Metric" (at 98.7552 46.99 0)
       (effects (font (size 1.27 1.27)) hide)
     )
@@
       (effects (font (size 1.27 1.27)) (justify left))
     )
-    (property "Footprint" "Resistor_SMD:R_0805_2012Metric_Pad1.20x1.40mm_HandSolder" (at 92.71 103.378 90)
+    (property "Footprint" "Resistor_SMD:R_0805_2012Metric" (at 92.71 103.378 90)
       (effects (font (size 1.27 1.27)) hide)
     )
@@
       (effects (font (size 1.27 1.27)) (justify left))
     )
-    (property "Footprint" "Resistor_SMD:R_0805_2012Metric_Pad1.20x1.40mm_HandSolder" (at 106.172 43.18 90)
+    (property "Footprint" "Resistor_SMD:R_0805_2012Metric" (at 106.172 43.18 90)
       (effects (font (size 1.27 1.27)) hide)
     )
@@
       (effects (font (size 1.27 1.27)) (justify left))
     )
-    (property "Footprint" "Resistor_SMD:R_0805_2012Metric_Pad1.20x1.40mm_HandSolder" (at 91.44 90.678 90)
+    (property "Footprint" "Resistor_SMD:R_0805_2012Metric" (at 91.44 90.678 90)
       (effects (font (size 1.27 1.27)) hide)
     )
@@
       (effects (font (size 1.27 1.27)))
     )
-    (property "Footprint" "LED_SMD:LED_0805_2012Metric_Pad1.15x1.40mm_HandSolder" (at 176.53 111.76 0)
+    (property "Footprint" "LED_SMD:LED_0805_2012Metric" (at 176.53 111.76 0)
       (effects (font (size 1.27 1.27)) hide)
     )
@@
       (effects (font (size 1.27 1.27)) (justify left))
     )
-    (property "Footprint" "Capacitor_SMD:C_0805_2012Metric_Pad1.18x1.45mm_HandSolder" (at 50.4952 144.78 0)
+    (property "Footprint" "Capacitor_SMD:C_0805_2012Metric" (at 50.4952 144.78 0)
       (effects (font (size 1.27 1.27)) hide)
     )
@@
       (effects (font (size 1.27 1.27)) (justify left))
     )
-    (property "Footprint" "Capacitor_SMD:C_0805_2012Metric_Pad1.18x1.45mm_HandSolder" (at 63.1952 144.78 0)
+    (property "Footprint" "Capacitor_SMD:C_0805_2012Metric" (at 63.1952 144.78 0)
       (effects (font (size 1.27 1.27)) hide)
     )
@@
       (effects (font (size 1.27 1.27)) (justify left))
     )
-    (property "Footprint" "Resistor_SMD:R_0805_2012Metric_Pad1.20x1.40mm_HandSolder" (at 50.292 67.31 90)
+    (property "Footprint" "Resistor_SMD:R_0805_2012Metric" (at 50.292 67.31 90)
       (effects (font (size 1.27 1.27)) hide)
     )
@@
       (effects (font (size 1.27 1.27)) (justify left))
     )
-    (property "Footprint" "Resistor_SMD:R_0805_2012Metric_Pad1.20x1.40mm_HandSolder" (at 91.44 85.598 90)
+    (property "Footprint" "Resistor_SMD:R_0805_2012Metric" (at 91.44 85.598 90)
       (effects (font (size 1.27 1.27)) hide)
     )
@@
       (effects (font (size 1.27 1.27)))
     )
-    (property "Footprint" "Resistor_SMD:R_0805_2012Metric_Pad1.20x1.40mm_HandSolder" (at 185.42 113.538 90)
-      (effects (font (size 1.27 1.27)) hide)
-    )
+    (property "Footprint" "Resistor_SMD:R_0805_2012Metric" (at 185.42 113.538 90)
+      (effects (font (size 1.27 1.27)) hide)
+    )
