File: Asignaciones/Room_Link/RELAY.kicad_sch (KiCad schematic)
At the start: 16 parts, among them K1 ADW11, K2 ADW11, K3 ADW11, K4 ADW11, K5 ADW11, U1 ULN2003A

Commit message: ROOM-LINK update KICAD
Parts:
- K1, K2, K3, K4, K5: footprint Relay_THT:Relay_1P1T_NO_10x24x18.8mm_Panasonic_ADW11xxxxW_THT -> nuevo simbolo:AZ921
- R1: value R -> 2.4K
- R2, R3, R4, R5: value R -> 1K
Changed lines of the file:
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@@
       (effects (font (size 1.27 1.27)) (justify left))
     )
-    (property "Footprint" "Relay_THT:Relay_1P1T_NO_10x24x18.8mm_Panasonic_ADW11xxxxW_THT" (at 211.455 53.34 0)
+    (property "Footprint" "nuevo simbolo:AZ921" (at 211.455 53.34 0)
       (effects (font (size 1.27 1.27)) hide)
     )
@@
       (effects (font (size 1.27 1.27)))
     )
-    (property "Value" "R" (at 142.24 105.41 90)
+    (property "Value" "2.4K" (at 142.24 105.41 90)
       (effects (font (size 1.27 1.27)))
     )
@@
       (effects (font (size 1.27 1.27)))
     )
-    (property "Value" "R" (at 106.68 102.87 90)
+    (property "Value" "1K" (at 106.68 102.87 90)
       (effects (font (size 1.27 1.27)))
     )
@@
       (effects (font (size 1.27 1.27)))
     )
-    (property "Value" "R" (at 190.5 107.95 90)
+    (property "Value" "1K" (at 190.5 107.95 90)
       (effects (font (size 1.27 1.27)))
     )
@@
       (effects (font (size 1.27 1.27)) (justify left))
     )
-    (property "Footprint" "Relay_THT:Relay_1P1T_NO_10x24x18.8mm_Panasonic_ADW11xxxxW_THT" (at 127.635 53.34 0)
+    (property "Footprint" "nuevo simbolo:AZ921" (at 127.635 53.34 0)
       (effects (font (size 1.27 1.27)) hide)
     )
@@
       (effects (font (size 1.27 1.27)) (justify left))
     )
-    (property "Footprint" "Relay_THT:Relay_1P1T_NO_10x24x18.8mm_Panasonic_ADW11xxxxW_THT" (at 163.195 53.34 0)
+    (property "Footprint" "nuevo simbolo:AZ921" (at 163.195 53.34 0)
       (effects (font (size 1.27 1.27)) hide)
     )
@@
       (effects (font (size 1.27 1.27)) (justify left))
     )
-    (property "Footprint" "Relay_THT:Relay_1P1T_NO_10x24x18.8mm_Panasonic_ADW11xxxxW_THT" (at 286.385 53.34 0)
+    (property "Footprint" "nuevo simbolo:AZ921" (at 286.385 53.34 0)
       (effects (font (size 1.27 1.27)) hide)
     )
@@
       (effects (font (size 1.27 1.27)))
     )
-    (property "Value" "R" (at 228.6 110.49 90)
+    (property "Value" "1K" (at 228.6 110.49 90)
       (effects (font (size 1.27 1.27)))
     )
@@
       (effects (font (size 1.27 1.27)) (justify left))
     )
-    (property "Footprint" "Relay_THT:Relay_1P1T_NO_10x24x18.8mm_Panasonic_ADW11xxxxW_THT" (at 248.285 53.34 0)
+    (property "Footprint" "nuevo simbolo:AZ921" (at 248.285 53.34 0)
       (effects (font (size 1.27 1.27)) hide)
     )
@@
       (effects (font (size 1.27 1.27)))
     )
-    (property "Value" "R" (at 265.43 114.3 90)
-      (effects (font (size 1.27 1.27)))
-    )
+    (property "Value" "1K" (at 265.43 114.3 90)
+      (effects (font (size 1.27 1.27)))
+    )

Commit message: Added nuevos cambios
Parts:
- removed K1, K2, K3, K4, K5: ADW11, nuevo simbolo:AZ921, symbol Relay:ADW11
- added U4, U6, U7, U8, U9: AZ921, nuevo simbolo:AZ921, symbol nuevos simvolos2:AZ921
- U1: footprint Package_DIP:DIP-16_W7.62mm_LongPads -> Package_SO:SOIC-16_3.9x9.9mm_P1.27mm
Connections:
- net +12V: now also U4.2, U6.2, U7.2, U8.2, U9.2
- net CON-FAN-C: now also U7.3, U8.3, U9.3
- net CON-FAN1: now also U7.4
- net CON-FAN2: now also U8.4
- net CON-FAN3: now also U9.4
- net CON-OUT1A: now also U4.4
- net CON-OUT1B: now also U4.3
- net CON-OUT2A: now also U6.4
- net CON-OUT2B: now also U6.3
- net at D2.1 (K), U1.14 (O3): now also U7.1
- net at D5.1 (K), U1.16 (O1): now also U4.1
- net at D4.1 (K), U1.12 (O5): now also U9.1
- net at D3.1 (K), U1.13 (O4): now also U8.1
- net at D1.1 (K), U1.15 (O2): now also U6.1

Commit message: Place component Added & routing
Parts:
- D1, D2, D3, D4, D5: footprint LED_SMD:LED_0805_2012Metric_Pad1.15x1.40mm_HandSolder -> LED_SMD:LED_0805_2012Metric
- R1, R2, R3, R4, R5: footprint Resistor_SMD:R_0805_2012Metric_Pad1.20x1.40mm_HandSolder -> Resistor_SMD:R_0805_2012Metric
Changed lines of the file:
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@@
       (effects (font (size 1.27 1.27)))
     )
-    (property "Footprint" "LED_SMD:LED_0805_2012Metric_Pad1.15x1.40mm_HandSolder" (at 95.25 106.68 0)
+    (property "Footprint" "LED_SMD:LED_0805_2012Metric" (at 95.25 106.68 0)
       (effects (font (size 1.27 1.27)) hide)
     )
@@
       (effects (font (size 1.27 1.27)))
     )
-    (property "Footprint" "Resistor_SMD:R_0805_2012Metric_Pad1.20x1.40mm_HandSolder" (at 142.24 110.998 90)
+    (property "Footprint" "Resistor_SMD:R_0805_2012Metric" (at 142.24 110.998 90)
       (effects (font (size 1.27 1.27)) hide)
     )
@@
       (effects (font (size 1.27 1.27)))
     )
-    (property "Footprint" "Resistor_SMD:R_0805_2012Metric_Pad1.20x1.40mm_HandSolder" (at 106.68 108.458 90)
+    (property "Footprint" "Resistor_SMD:R_0805_2012Metric" (at 106.68 108.458 90)
       (effects (font (size 1.27 1.27)) hide)
     )
@@
       (effects (font (size 1.27 1.27)))
     )
-    (property "Footprint" "Resistor_SMD:R_0805_2012Metric_Pad1.20x1.40mm_HandSolder" (at 190.5 113.538 90)
+    (property "Footprint" "Resistor_SMD:R_0805_2012Metric" (at 190.5 113.538 90)
       (effects (font (size 1.27 1.27)) hide)
     )
@@
       (effects (font (size 1.27 1.27)))
     )
-    (property "Footprint" "LED_SMD:LED_0805_2012Metric_Pad1.15x1.40mm_HandSolder" (at 254 118.11 0)
+    (property "Footprint" "LED_SMD:LED_0805_2012Metric" (at 254 118.11 0)
       (effects (font (size 1.27 1.27)) hide)
     )
@@
       (effects (font (size 1.27 1.27)))
     )
-    (property "Footprint" "LED_SMD:LED_0805_2012Metric_Pad1.15x1.40mm_HandSolder" (at 217.17 114.3 0)
+    (property "Footprint" "LED_SMD:LED_0805_2012Metric" (at 217.17 114.3 0)
       (effects (font (size 1.27 1.27)) hide)
     )
@@
       (effects (font (size 1.27 1.27)))
     )
-    (property "Footprint" "Resistor_SMD:R_0805_2012Metric_Pad1.20x1.40mm_HandSolder" (at 228.6 116.078 90)
+    (property "Footprint" "Resistor_SMD:R_0805_2012Metric" (at 228.6 116.078 90)
       (effects (font (size 1.27 1.27)) hide)
     )
@@
       (effects (font (size 1.27 1.27)))
     )
-    (property "Footprint" "LED_SMD:LED_0805_2012Metric_Pad1.15x1.40mm_HandSolder" (at 130.81 109.22 0)
+    (property "Footprint" "LED_SMD:LED_0805_2012Metric" (at 130.81 109.22 0)
       (effects (font (size 1.27 1.27)) hide)
     )
@@
       (effects (font (size 1.27 1.27)))
     )
-    (property "Footprint" "Resistor_SMD:R_0805_2012Metric_Pad1.20x1.40mm_HandSolder" (at 265.43 119.888 90)
+    (property "Footprint" "Resistor_SMD:R_0805_2012Metric" (at 265.43 119.888 90)
       (effects (font (size 1.27 1.27)) hide)
     )
@@
       (effects (font (size 1.27 1.27)))
     )
-    (property "Footprint" "LED_SMD:LED_0805_2012Metric_Pad1.15x1.40mm_HandSolder" (at 179.07 111.76 0)
-      (effects (font (size 1.27 1.27)) hide)
-    )
+    (property "Footprint" "LED_SMD:LED_0805_2012Metric" (at 179.07 111.76 0)
+      (effects (font (size 1.27 1.27)) hide)
+    )
