File: Asignaciones/Room_Link/Room_Link.kicad_pcb (KiCad board)
At the start: 2 copper layers, 0 parts

Commit message: Added new changes ROOM-LINK
Parts:
- added C1: 0.1uF, Capacitor_SMD:C_0805_2012Metric_Pad1.18x1.45mm_HandSolder, F.Cu at (-38.1, 35.5)
- added C10: 0.1uF, Capacitor_SMD:C_0805_2012Metric_Pad1.18x1.45mm_HandSolder, F.Cu at (-122.8, 5.66)
- added C11: 22 uF, Capacitor_SMD:C_0805_2012Metric_Pad1.18x1.45mm_HandSolder, F.Cu at (-122.8, 8.66)
- added C12: 0.1uF, Capacitor_SMD:C_0805_2012Metric_Pad1.18x1.45mm_HandSolder, F.Cu at (-122.8, 11.7)
- added C2: 0.1uF, Capacitor_SMD:C_0805_2012Metric_Pad1.18x1.45mm_HandSolder, F.Cu at (-38.1, 38.5)
- added C3: 0.1uF, Capacitor_SMD:C_0805_2012Metric_Pad1.18x1.45mm_HandSolder, F.Cu at (-38.1, 41.5)
- added C4: 0.1uF, Capacitor_SMD:C_0805_2012Metric_Pad1.18x1.45mm_HandSolder, F.Cu at (-38.1, 44.5)
- added C5: 1 uF, Capacitor_SMD:C_0805_2012Metric_Pad1.18x1.45mm_HandSolder, F.Cu at (-32.0, 56.1)
- added C6: 0.1 uF, Capacitor_SMD:C_0805_2012Metric_Pad1.18x1.45mm_HandSolder, F.Cu at (-32.0, 59.1)
- added C7: 0.1uF 25v, Capacitor_SMD:C_0805_2012Metric_Pad1.18x1.45mm_HandSolder, F.Cu at (-94.9, 57.1)
- added C8: 0.1uF 25v, Capacitor_SMD:C_0805_2012Metric_Pad1.18x1.45mm_HandSolder, F.Cu at (-94.9, 60.1)
- added C9: 47uF 10, Capacitor_SMD:C_0805_2012Metric_Pad1.18x1.45mm_HandSolder, F.Cu at (-94.9, 63.1)
- added D1: LED, LED_SMD:LED_0805_2012Metric_Pad1.15x1.40mm_HandSolder, F.Cu at (-51.7, 39.7)
- added D10: LED, LED_SMD:LED_0805_2012Metric_Pad1.15x1.40mm_HandSolder, F.Cu at (-54.4, 72.9)
- added D11: SM712-02HTG, sm712:SM71202HTG, F.Cu at (-59.8, 74.5)
- added D12: SMBJ12CA, nuevo simbolo:SMBJ12CA, F.Cu at (-72.1, 74.1)
- added D13: LED, LED_SMD:LED_0805_2012Metric_Pad1.15x1.40mm_HandSolder, F.Cu at (-104.4, 57.1)
- added D14: SMBJ12CA, nuevo simbolo:SMBJ12CA, F.Cu at (-29.1, 50.9)
- added D15: SM712-02HTG, sm712:SM71202HTG, F.Cu at (-37.5, 57.6)
- added D16: LED, LED_SMD:LED_0805_2012Metric_Pad1.15x1.40mm_HandSolder, F.Cu at (-104.4, 60.2)
- added D17: LED, LED_SMD:LED_0805_2012Metric_Pad1.15x1.40mm_HandSolder, F.Cu at (-104.4, 63.2)
- added D18: LED, LED_SMD:LED_0805_2012Metric_Pad1.15x1.40mm_HandSolder, F.Cu at (-104.4, 66.3)
- added D19: LED, LED_SMD:LED_0805_2012Metric_Pad1.15x1.40mm_HandSolder, F.Cu at (-117.9, 14.1)
- added D2: LED, LED_SMD:LED_0805_2012Metric_Pad1.15x1.40mm_HandSolder, F.Cu at (-51.7, 42.7)
- added D3: LED, LED_SMD:LED_0805_2012Metric_Pad1.15x1.40mm_HandSolder, F.Cu at (-51.7, 45.8)
- added D4: LED, LED_SMD:LED_0805_2012Metric_Pad1.15x1.40mm_HandSolder, F.Cu at (-51.7, 48.8)
- added D5: LED, LED_SMD:LED_0805_2012Metric_Pad1.15x1.40mm_HandSolder, F.Cu at (-51.7, 51.9)
- added D6: LED, LED_SMD:LED_0805_2012Metric_Pad1.15x1.40mm_HandSolder, F.Cu at (-33.2, 35.5)
- added D7: LED, LED_SMD:LED_0805_2012Metric_Pad1.15x1.40mm_HandSolder, F.Cu at (-33.2, 38.5)
- added D8: LED, LED_SMD:LED_0805_2012Metric_Pad1.15x1.40mm_HandSolder, F.Cu at (-33.2, 41.6)
- added D9: LED, LED_SMD:LED_0805_2012Metric_Pad1.15x1.40mm_HandSolder, F.Cu at (-33.2, 44.6)
- added F1: PTS120660V010, PTS12066V050:FUSC3216X68N, F.Cu at (-65.7, 73.1)
- added F2: PTS120660V010, PTS12066V050:FUSC3216X68N, F.Cu at (-65.7, 76.4)
- added F3: PTS120660V010, PTS12066V050:FUSC3216X68N, F.Cu at (-120.4, 76.8)
- added IC1: LM1117T-3.3, lm1117:TO254P470X1016X2222-3P, F.Cu at (-114.9, 71.7)
- added J1: TBP04R12-500-02BE, TBP04R12-500-02BE:CUI_TBP04R12-500-02BE, F.Cu at (-71.7, 3.52)
- added J2: TBP04R12-500-03BE, TBP04R12-500-03BE:CUI_TBP04R12-500-03BE, F.Cu at (-32.8, 3.52)
- added J3: TBP04R12-500-08BE, TBP04R12-500-08BE:CUI_TBP04R12-500-08BE, F.Cu at (-71.7, -25.4)
- added J4: TBP04R12-500-08BE, TBP04R12-500-08BE:CUI_TBP04R12-500-08BE, F.Cu at (-71.7, -11.0)
- added J5: TBP04R12-500-02BE, TBP04R12-500-02BE:CUI_TBP04R12-500-02BE, F.Cu at (-58.7, 3.52)
- added J6: TBP04R12-500-02BE, TBP04R12-500-02BE:CUI_TBP04R12-500-02BE, F.Cu at (-45.8, 3.52)
- added J8: Screw_Terminal_01x06, Connector_PinHeader_2.54mm:PinHeader_2x06_P2.54mm_Vertical_SMD, F.Cu at (-131.6, 12.8)
- added J9: Conn_ARM_JTAG_SWD_10, Connector_PinHeader_1.27mm:PinHeader_2x05_P1.27mm_Vertical, F.Cu at (-118.2, 5.83)
- added K1: ADW11, nuevo simbolo:AZ921, F.Cu at (-67.0, 22.2)
- added K2: ADW11, nuevo simbolo:AZ921, F.Cu at (-67.0, 28.9)
- added K3: ADW11, nuevo simbolo:AZ921, F.Cu at (-67.0, 35.6)
- added K4: ADW11, nuevo simbolo:AZ921, F.Cu at (-67.0, 42.2)
- added K5: ADW11, nuevo simbolo:AZ921, F.Cu at (-67.0, 48.9)
- added PS1: HLK-PM12, KiCad:HLKPM12, F.Cu at (-127.6, 41.6)
- added PS2: B0505S-W2R2, B0505S:B0505SW2R2, F.Cu at (-103.3, 74.4)
- added Q1: FODM2705, nuevo simbolo:FODM2705, F.Cu at (-22.0, 18.4)
- added Q2: FODM2705, nuevo simbolo:FODM2705, F.Cu at (-22.0, 23.3)
- added Q3: FODM2705, nuevo simbolo:FODM2705, F.Cu at (-22.0, 28.1)
- added Q4: FODM2705, nuevo simbolo:FODM2705, F.Cu at (-22.0, 33.0)
- added R1: 2.4K, Resistor_SMD:R_0805_2012Metric_Pad1.20x1.40mm_HandSolder, F.Cu at (-46.9, 39.7)
- added R10: 10, Resistor_SMD:R_0805_2012Metric_Pad1.20x1.40mm_HandSolder, F.Cu at (-38.1, 29.6)
- added R11: 470, Resistor_SMD:R_0805_2012Metric_Pad1.20x1.40mm_HandSolder, F.Cu at (-38.1, 32.5)
- added R12: 10k, Resistor_SMD:R_0805_2012Metric_Pad1.20x1.40mm_HandSolder, F.Cu at (-33.4, 17.8)
- added R13: 470, Resistor_SMD:R_0805_2012Metric_Pad1.20x1.40mm_HandSolder, F.Cu at (-33.4, 20.7)
- added R14: 330, Resistor_SMD:R_0805_2012Metric_Pad1.20x1.40mm_HandSolder, F.Cu at (-33.4, 23.7)
- added R15: 10, Resistor_SMD:R_0805_2012Metric_Pad1.20x1.40mm_HandSolder, F.Cu at (-33.4, 26.6)
- added R16: 10k, Resistor_SMD:R_0805_2012Metric_Pad1.20x1.40mm_HandSolder, F.Cu at (-33.4, 29.6)
- added R17: 470, Resistor_SMD:R_0805_2012Metric_Pad1.20x1.40mm_HandSolder, F.Cu at (-33.4, 32.5)
- added R18: 330, Resistor_SMD:R_0805_2012Metric_Pad1.20x1.40mm_HandSolder, F.Cu at (-28.6, 17.8)
- added R19: 10, Resistor_SMD:R_0805_2012Metric_Pad1.20x1.40mm_HandSolder, F.Cu at (-28.6, 20.7)
- added R2: 1K, Resistor_SMD:R_0805_2012Metric_Pad1.20x1.40mm_HandSolder, F.Cu at (-46.9, 42.6)
- added R20: 10k, Resistor_SMD:R_0805_2012Metric_Pad1.20x1.40mm_HandSolder, F.Cu at (-28.6, 23.7)
- added R21: 470, Resistor_SMD:R_0805_2012Metric_Pad1.20x1.40mm_HandSolder, F.Cu at (-28.6, 26.6)
- added R22: 2.2k, Resistor_SMD:R_0805_2012Metric_Pad1.20x1.40mm_HandSolder, F.Cu at (-53.9, 56.9)
- added R23: 2.2k, Resistor_SMD:R_0805_2012Metric_Pad1.20x1.40mm_HandSolder, F.Cu at (-53.9, 59.8)
- added R24: 2.2k, Resistor_SMD:R_0805_2012Metric_Pad1.20x1.40mm_HandSolder, F.Cu at (-53.9, 62.8)
- added R25: 10, Resistor_SMD:R_0805_2012Metric_Pad1.20x1.40mm_HandSolder, F.Cu at (-53.9, 65.7)
- added R26: 10, Resistor_SMD:R_0805_2012Metric_Pad1.20x1.40mm_HandSolder, F.Cu at (-53.9, 68.7)
- added R27: 10, Resistor_SMD:R_0805_2012Metric_Pad1.20x1.40mm_HandSolder, F.Cu at (-27.3, 56.0)
- added R28: 10 1%, Resistor_SMD:R_0805_2012Metric_Pad1.20x1.40mm_HandSolder, F.Cu at (-27.3, 59.0)
- added R29: 10, Resistor_SMD:R_0805_2012Metric_Pad1.20x1.40mm_HandSolder, F.Cu at (-27.3, 61.9)
- added R3: 1K, Resistor_SMD:R_0805_2012Metric_Pad1.20x1.40mm_HandSolder, F.Cu at (-46.9, 45.6)
- added R30: R, Resistor_SMD:R_0805_2012Metric_Pad1.20x1.40mm_HandSolder, F.Cu at (-99.7, 57.1)
- added R31: 2.2k, Resistor_SMD:R_0805_2012Metric_Pad1.20x1.40mm_HandSolder, F.Cu at (-99.7, 60.0)
- added R32: 470, Resistor_SMD:R_0805_2012Metric_Pad1.20x1.40mm_HandSolder, F.Cu at (-99.7, 63.0)
- added R33: 1k, Resistor_SMD:R_0805_2012Metric_Pad1.20x1.40mm_HandSolder, F.Cu at (-99.7, 65.9)
- added R34: 22k, Resistor_SMD:R_0805_2012Metric_Pad1.20x1.40mm_HandSolder, F.Cu at (-86.6, -36.7)
- added R35: 1k, Resistor_SMD:R_0805_2012Metric_Pad1.20x1.40mm_HandSolder, F.Cu at (-86.6, -33.7)
- added R36: 100k, Resistor_SMD:R_0805_2012Metric_Pad1.20x1.40mm_HandSolder, F.Cu at (-86.6, -30.8)
- added R37: 100k, Resistor_SMD:R_0805_2012Metric_Pad1.20x1.40mm_HandSolder, F.Cu at (-86.6, -27.8)
- added R38: 100k, Resistor_SMD:R_0805_2012Metric_Pad1.20x1.40mm_HandSolder, F.Cu at (-86.6, -24.9)
- added R39: 100k, Resistor_SMD:R_0805_2012Metric_Pad1.20x1.40mm_HandSolder, F.Cu at (-86.6, -21.9)
- added R4: 1K, Resistor_SMD:R_0805_2012Metric_Pad1.20x1.40mm_HandSolder, F.Cu at (-46.9, 48.5)
- added R40: 100k, Resistor_SMD:R_0805_2012Metric_Pad1.20x1.40mm_HandSolder, F.Cu at (-86.6, -19.0)
- added R41: 470, Resistor_SMD:R_0805_2012Metric_Pad1.20x1.40mm_HandSolder, F.Cu at (-86.6, -16.0)
- added R5: 1K, Resistor_SMD:R_0805_2012Metric_Pad1.20x1.40mm_HandSolder, F.Cu at (-46.9, 51.5)
- added R6: 10k, Resistor_SMD:R_0805_2012Metric_Pad1.20x1.40mm_HandSolder, F.Cu at (-38.1, 17.8)
- added R7: 330, Resistor_SMD:R_0805_2012Metric_Pad1.20x1.40mm_HandSolder, F.Cu at (-38.1, 20.7)
- added R8: 330, Resistor_SMD:R_0805_2012Metric_Pad1.20x1.40mm_HandSolder, F.Cu at (-38.1, 23.7)
- added R9: 10, Resistor_SMD:R_0805_2012Metric_Pad1.20x1.40mm_HandSolder, F.Cu at (-38.1, 26.6)
- added RV1: MOVTP20V275N, movtp:MOVTP20V275N, F.Cu at (-122.9, 62.5)
- added U1: ULN2003A, Package_DIP:DIP-16_W7.62mm_LongPads, F.Cu at (-52.1, 18.4)
- added U2: TD521D485H-E, nuevo simbolo:TD521D485H-E, F.Cu at (-65.9, 63.2)
- added U3: SP485ECN-L, footprints:NSOIC-8-L, F.Cu at (-36.5, 51.4)
- added U5: ESP32-WROOM-32, RF_Module:ESP32-WROOM-32, F.Cu at (-113.5, -6.88)
- added Z1: 1SMA5918BT3G, huellas:DIOM5226X220N, F.Cu at (-127.3, 71.5)
- added Z2: 1SMA5918BT3G, huellas:DIOM5226X220N, F.Cu at (-127.3, 76.0)

Commit message: Added nuevos cambios
Parts:
- removed K1, K2, K3, K4, K5: ADW11, nuevo simbolo:AZ921
- removed PS2: B0505S-W2R2, B0505S:B0505SW2R2
- added U10: B0505XT-2WR2, nuevo simbolo:B0505S-W2R2, F.Cu at (182.5, 125.1)
- added U4: AZ921, nuevo simbolo:AZ921, F.Cu at (174.6, 69.2)
- added U6: AZ921, nuevo simbolo:AZ921, F.Cu at (181.3, 69.2)
- added U7: AZ921, nuevo simbolo:AZ921, F.Cu at (153.2, 69.2)
- added U8: AZ921, nuevo simbolo:AZ921, F.Cu at (160.7, 69.2)
- added U9: AZ921, nuevo simbolo:AZ921, F.Cu at (167.4, 69.2)
- C9: footprint Capacitor_SMD:C_0805_2012Metric_Pad1.18x1.45mm_HandSolder -> Capacitor_SMD:CP_Elec_6.3x5.7
- F3: footprint PTS12066V050:FUSC3216X68N -> Fuse:Fuseholder_Cylinder-5x20mm_Stelvio-Kontek_PTF78_Horizontal_Open
- J8: footprint Connector_PinHeader_2.54mm:PinHeader_2x06_P2.54mm_Vertical_SMD -> Connector_PinHeader_2.54mm:PinHeader_1x06_P2.54mm_Vertical_SMD_Pin1Left
- J9: value Conn_ARM_JTAG_SWD_10 -> JTAG_ ESP32
- R35: value 1k -> 22k
- R36, R37, R38, R39, R40: value 100k -> 10K
- U1: footprint Package_DIP:DIP-16_W7.62mm_LongPads -> Package_SO:SOIC-16_3.9x9.9mm_P1.27mm
- moved J8 322.2 mm to (175.7, 109.8), turned to -90 degrees
- moved U5 305.0 mm to (174.9, 92.5), turned to -90 degrees
- moved J3 272.1 mm to (189.0, 52.5), turned to 180 degrees
- moved J4 266.3 mm to (154.0, 130.5)
- moved D19 258.8 mm to (134.5, 71.0), turned to -90 degrees
- moved J9 252.5 mm to (124.2, 76.4)
- moved R35 252.0 mm to (145.5, 64.5), turned to 90 degrees
- moved R36 248.0 mm to (144.0, 60.5), turned to 90 degrees
- moved R37 246.2 mm to (142.0, 63.5), turned to 180 degrees
- moved R38 241.4 mm to (138.0, 63.5), turned to 180 degrees
- moved R34 238.8 mm to (129.0, 66.0), turned to 90 degrees
- moved R39 236.6 mm to (134.0, 63.5), turned to 180 degrees
- moved PS1 236.1 mm to (101.0, 100.7), turned to 90 degrees
- moved F3 235.2 mm to (108.5, 131.1), turned to 90 degrees
- moved R41 234.4 mm to (131.0, 71.0), turned to 90 degrees
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Connections:
- net MTCLK renamed MTCK
- net MTD1 renamed MTDI
- U5 pad 13: MTM5 -> MTMS
- U5 pad 25: /Room-Link/CONTROL/INPUT_1MICRO -> /Room-Link/CONTROL/INPUT_3MICRO
- U5 pad 26: /Room-Link/CONTROL/INPUT_3MICRO -> /Room-Link/CONTROL/INPUT_2MICRO
- U5 pad 29: /Room-Link/CONTROL/INPUT_2MICRO -> /Room-Link/CONTROL/INPUT_1MICRO

Commit message: new changes added
Parts:
- C9: footprint Capacitor_SMD:CP_Elec_6.3x5.7 -> Capacitor_SMD:C_0805_2012Metric_Pad1.18x1.45mm_HandSolder
- RV1: footprint movtp:MOVTP20V275N -> B722:B72210S1140K501
- moved C10 207.3 mm to (121.0, 66.0), turned to 90 degrees
- moved C1 195.1 mm to (143.5, 143.0)
- moved R7 193.2 mm to (133.0, 143.0)
- moved F2 166.6 mm to (107.0, 177.0)
- moved D11 164.6 mm to (99.0, 173.5), turned to -90 degrees
- moved R26 164.1 mm to (102.5, 177.0)
- moved D12 163.0 mm to (94.0, 173.5)
- moved D10 162.3 mm to (98.5, 177.0), turned to 180 degrees
- moved R25 146.1 mm to (95.0, 168.0)
- moved F1 145.7 mm to (99.5, 168.0)
- moved D14 136.4 mm to (123.5, 58.0), turned to -90 degrees
- moved R22 134.1 mm to (68.5, 145.6)
- moved R23 134.1 mm to (68.5, 148.5)
- moved IC1 107.4 mm to (207.5, 122.0)
- moved D15 106.2 mm to (94.5, 60.9), turned to 180 degrees
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
Commit message: Place component Added & routing
Parts:
- removed U10: B0505XT-2WR2, nuevo simbolo:B0505S-W2R2
- added PS2: B0505S-W2R2, B0505S:B0505SW2R2, F.Cu at (189.5, 123.0)
- C10, C11, C12, C4, C5, C6, C7, C8, C9: footprint Capacitor_SMD:C_0805_2012Metric_Pad1.18x1.45mm_HandSolder -> Capacitor_SMD:C_0805_2012Metric
- D1, D10, D13, D16, D17, D18, D19, D2, D3, D4, D5, D6, D7, D8, D9: footprint LED_SMD:LED_0805_2012Metric_Pad1.15x1.40mm_HandSolder -> LED_SMD:LED_0805_2012Metric
- D11, D15: footprint sm712:SM71202HTG -> Package_TO_SOT_SMD:SOT-23
- R1, R10, R11, R12, R13, R14, R15, R16, R17, R18, R19, R2, R20, R21, R22, R23, R24, R25, R26, R27, R28, R29, R3, R30, R31, R32, R33, R34, R35, R36, R37, R38, R39, R4, R40, R41, R5, R6, R7, R8, R9: footprint Resistor_SMD:R_0805_2012Metric_Pad1.20x1.40mm_HandSolder -> Resistor_SMD:R_0805_2012Metric
- Z1, Z2: footprint huellas:DIOM5226X220N -> Diode_SMD:D_SMB
- moved Z2 257.1 mm to (188.5, 119.5)
- moved C11 256.6 mm to (182.4, 81.0), turned to 0 degrees
- moved D13 254.2 mm to (183.5, 120.1)
- moved C12 252.0 mm to (182.5, 79.0), turned to 0 degrees
- moved R30 249.1 mm to (183.0, 115.0), turned to 0 degrees
- moved D17 230.7 mm to (125.5, 66.5)
- moved R32 226.5 mm to (125.5, 69.0), turned to 0 degrees
- moved R10 221.4 mm to (178.5, 120.5), turned to 0 degrees
- moved R12 218.6 mm to (178.5, 115.0)
- moved D6 217.6 mm to (168.9, 108.0), turned to 180 degrees
- moved R11 217.2 mm to (169.0, 110.5), turned to 180 degrees
- moved R13 216.8 mm to (178.6, 112.5)
- moved Z1 215.0 mm to (120.8, 78.0), turned to 0 degrees
- moved R6 213.5 mm to (169.0, 113.0), turned to 180 degrees
- moved C8 213.3 mm to (121.5, 74.5), turned to 180 degrees
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Connections:
- C5 pad 1: +5V -> VDD
- C6 pad 1: +5V -> VDD
- C7 pad 2: GND -> +12V
- C8 pad 1: +3.3V -> VDD
- C8 pad 2: GND -> +12V
- C9 pad 1: +3.3V -> VDD
- C9 pad 2: GND -> +12V
- D16 pad 1: GND -> +12V
- D17 pad 1: GND -> +12V
- D18 pad 1: GND -> +12V
- IC1 pad 1: GND -> +12V
- IC1 pad 2: +3.3V -> VDD
- J3 pad 1: /Room-Link/CON-OUT2A -> /Room-Link/CON-OUT2B
- J3 pad 2: /Room-Link/CON-OUT2B -> /Room-Link/CON-OUT2A
- J5 pad 2: GND -> +12V
- PS1 pad 3: GND -> +12V
- PS1 pad 4: GND -> +12V
- R11 pad 1: +5V -> VDD
- R12 pad 1: +5V -> VDD
- R13 pad 1: +5V -> VDD
- R14 pad 1: VDD -> +3.3V
- R16 pad 1: +5V -> VDD
- R17 pad 1: +5V -> VDD
- R18 pad 1: VDD -> +3.3V
- R20 pad 1: +5V -> VDD
- R21 pad 1: +5V -> VDD
- R6 pad 1: +5V -> VDD
- R7 pad 1: VDD -> +3.3V
- R8 pad 1: VDD -> +3.3V
- U2 pad 2: +5V -> VDD
- U3 pad 8: +5V -> VDD
- Z1 pad 1: GND -> +12V
- Z1 pad 2: +3.3V -> VDD
- Z2 pad 2: VDD -> +3.3V
Routing:
- net /Room-Link/CONTROL/RLY_OUT2_MICRO: track 0.00 -> 72.2 mm
- net /Room-Link/CONTROL/RLY_OUT1_MICRO: track 0.00 -> 67.1 mm
- net Net-(D4-K): track 0.00 -> 56.4 mm
- net MTD0: track 0.00 -> 36.7 mm
- net Net-(D5-K): track 0.00 -> 36.5 mm
- net Net-(PS1-AC_2): track 0.00 -> 35.3 mm
- net /Room-Link/CON-NEUT: track 0.00 -> 35.0 mm
- net +12V: track 0.00 -> 34.2 mm
- net Net-(U3-B): track 0.00 -> 32.3 mm
- net Net-(U3-A): track 0.00 -> 27.7 mm
- net /Room-Link/CON-FAN-C: track 0.00 -> 23.5 mm
- net /Room-Link/CON-L1: track 0.00 -> 22.0 mm
- net MTCK: track 0.00 -> 19.2 mm
- net Net-(D1-K): track 0.00 -> 19.1 mm
- net /Room-Link/CON-OUT2B: track 0.00 -> 16.4 mm
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
Commit message: Terminado'disque'
Parts:
- J8: footprint Connector_PinHeader_2.54mm:PinHeader_1x06_P2.54mm_Vertical_SMD_Pin1Left -> Connector_PinHeader_2.54mm:PinHeader_2x03_P2.54mm_Vertical
- moved Z1 0.82 mm to (121.5, 78.5)
- moved C2 0.50 mm to (178.5, 118.0)
- moved C10 0.50 mm to (176.5, 79.5)
- moved C8 0.50 mm to (121.5, 75.0)
- moved Q2 0.50 mm to (174.0, 113.5)
- moved R34 0.50 mm to (176.5, 81.5)
Connections:
- C7 pad 2: +12V -> GND
- C8 pad 2: +12V -> GND
- D17 pad 1: +12V -> GND
- IC1 pad 1: +12V -> GND
- PS2 pad 1: +12V -> GND
- R33 pad 1: /Room-Link/CON-DC+ -> unconnected-(R33-Pad1)
- Z1 pad 1: +12V -> GND
Routing:
- net VDD: track 0.00 -> 224.2 mm, vias 0 -> 15
- net +3.3V: track 0.00 -> 114.3 mm, vias 0 -> 4
- net +12V: track 34.2 -> 142.1 mm, vias 0 -> 4
- net /Room-Link/CONTROL/Tx_RS485_LCD: track 0.00 -> 98.9 mm, vias 0 -> 2
- net /Room-Link/CONTROL/Rx_RS485_eXT: track 0.00 -> 88.4 mm, vias 0 -> 2
- net /Room-Link/CONTROL/Rx_RS485_lcd: track 0.00 -> 84.7 mm, vias 0 -> 2
- net /Room-Link/CONTROL/COM_RS485_LCD: track 0.00 -> 80.5 mm, vias 0 -> 2
- net /Room-Link/CONTROL/RLY_FAN2_MICRO: track 0.00 -> 80.2 mm, vias 0 -> 2
- net /Room-Link/CONTROL/CON_RS485_eXT: track 0.00 -> 74.8 mm, vias 0 -> 2
- net /Room-Link/CONTROL/Tx_RS485_eXT: track 0.00 -> 61.5 mm, vias 0 -> 2
- net /Room-Link/CON-IN1+: track 0.00 -> 54.9 mm, vias 0 -> 1
- net EN: track 8.53 -> 57.3 mm, vias 0 -> 4
- net Net-(D1-K): track 19.1 -> 67.7 mm, vias 0 -> 1
- net /Room-Link/CONTROL/RLY_FAN1_MICRO: track 0.00 -> 47.0 mm, vias 0 -> 2
- net Net-(D3-K): track 0.00 -> 42.5 mm, vias 0 -> 2
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- added copper zone on B.Cu, net Earth
- added copper zone on In1.Cu, net GND
Other:
- copper layers 2 -> 4
