File: Asignaciones/Room_Link/Room_Link.kicad_sch (KiCad schematic)
At the start: 6 parts, among them J1 TBP04R12-500-02BE, J2 TBP04R12-500-03BE, J3 TBP04R12-500-08BE, J4 TBP04R12-500-08BE, J5 TBP04R12-500-02BE, J6 TBP04R12-500-02BE

Commit message: Nuevos cambios del Room-Link
Other:
- moved on the sheet: J2, J4, J6

Commit message: ROOM-LINK update KICAD
Parts:
- J1, J5, J6: footprint CUI_TBP04R12-500-02BE -> TBP04R12-500-02BE:CUI_TBP04R12-500-02BE
- J2: footprint CUI_TBP04R12-500-03BE -> TBP04R12-500-03BE:CUI_TBP04R12-500-03BE
- J3, J4: footprint CUI_TBP04R12-500-08BE -> TBP04R12-500-08BE:CUI_TBP04R12-500-08BE
Changed lines of the file:
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@@
       (effects (font (size 1.27 1.27)) (justify left))
     )
-    (property "Footprint" "CUI_TBP04R12-500-03BE" (at 113.03 111.76 0)
+    (property "Footprint" "TBP04R12-500-03BE:CUI_TBP04R12-500-03BE" (at 113.03 111.76 0)
       (effects (font (size 1.27 1.27)) (justify left bottom) hide)
     )
@@
       (effects (font (size 1.27 1.27)) (justify right))
     )
-    (property "Footprint" "CUI_TBP04R12-500-02BE" (at 92.71 53.34 0)
+    (property "Footprint" "TBP04R12-500-02BE:CUI_TBP04R12-500-02BE" (at 92.71 53.34 0)
       (effects (font (size 1.27 1.27)) (justify left bottom) hide)
     )
@@
       (effects (font (size 1.27 1.27)) (justify left))
     )
-    (property "Footprint" "CUI_TBP04R12-500-08BE" (at 167.64 111.76 0)
+    (property "Footprint" "TBP04R12-500-08BE:CUI_TBP04R12-500-08BE" (at 167.64 111.76 0)
       (effects (font (size 1.27 1.27)) (justify left bottom) hide)
     )
@@
       (effects (font (size 1.27 1.27)) (justify right))
     )
-    (property "Footprint" "CUI_TBP04R12-500-08BE" (at 165.1 53.34 0)
+    (property "Footprint" "TBP04R12-500-08BE:CUI_TBP04R12-500-08BE" (at 165.1 53.34 0)
       (effects (font (size 1.27 1.27)) (justify left bottom) hide)
     )
@@
       (effects (font (size 1.27 1.27)) (justify left))
     )
-    (property "Footprint" "CUI_TBP04R12-500-02BE" (at 91.44 111.76 0)
+    (property "Footprint" "TBP04R12-500-02BE:CUI_TBP04R12-500-02BE" (at 91.44 111.76 0)
       (effects (font (size 1.27 1.27)) (justify left bottom) hide)
     )
@@
       (effects (font (size 1.27 1.27)) (justify right))
     )
-    (property "Footprint" "CUI_TBP04R12-500-02BE" (at 107.95 53.34 0)
+    (property "Footprint" "TBP04R12-500-02BE:CUI_TBP04R12-500-02BE" (at 107.95 53.34 0)
       (effects (font (size 1.27 1.27)) (justify left bottom) hide)
     )

Commit message: Terminado'disque'
Connections:
- net Room-Link/CON-OUT2A: now also J3.2; no longer J3.1
- net Room-Link/CON-OUT2B: now also J3.1; no longer J3.2
Changed lines of the file:
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@@
+    (stroke (width 0) (type default))
+  )
+  (wire (pts (xy 157.48 63.5) (xy 157.48 67.31))
     (stroke (width 0) (type default))
   )
@@
     (stroke (width 0) (type default))
   )
+  (wire (pts (xy 160.02 63.5) (xy 160.02 67.31))
+    (stroke (width 0) (type default))
+  )
   (wire (pts (xy 172.72 63.5) (xy 172.72 67.31))
     (stroke (width 0) (type default))
@@
     (stroke (width 0) (type default))
   )
-  (wire (pts (xy 160.02 63.5) (xy 160.02 67.31))
-    (stroke (width 0) (type default))
-  )
   (wire (pts (xy 160.02 96.52) (xy 160.02 101.6))
     (stroke (width 0) (type default))
   )
   (wire (pts (xy 167.64 63.5) (xy 167.64 67.31))
-    (stroke (width 0) (type default))
-  )
-  (wire (pts (xy 157.48 63.5) (xy 157.48 67.31))
     (stroke (width 0) (type default))
   )
@@
       (effects (font (size 1.27 1.27)) (justify left))
     )
-    (pin "CON-OUT2A" input (at 157.48 67.31 90)
-      (effects (font (size 1.27 1.27)) (justify right))
-    )
-    (pin "CON-OUT2B" input (at 160.02 67.31 90)
-      (effects (font (size 1.27 1.27)) (justify right))
-    )
+    (pin "CON-OUT2A" input (at 160.02 67.31 90)
+      (effects (font (size 1.27 1.27)) (justify right))
+    )
+    (pin "CON-OUT2B" input (at 157.48 67.31 90)
+      (effects (font (size 1.27 1.27)) (justify right))
+    )
